Commit message: fixed config and params and not bit is behaving as intended

File: src/urdf/diff_lidar.urdf (robot description, URDF)
Before this commit: robot diff_lidar, 9 links, 8 joints
Joints:
- joint camera_joint: origin xyz=0.15 0 0.15 rpy=0 0 0 -> xyz=0.325 0 0.1 rpy=0 0 0
- joint gps_joint: origin xyz=0 0 0.12 -> xyz=-0.1 0 0.21 rpy=0 0 0
- joint imu_joint: origin xyz=0 0 0.2 -> xyz=0.1 0 0.205 rpy=0 0 0
